File: SOS-Water-Ingress-Sensor.brd (EAGLE design)
At the start: 25.4 x 13 mm, 12 parts

Commit message: Minor tweaks to layout all around.
Parts:
- moved U$7 0.16 mm to (24.3, 0.95)
Connections:
- net GND: now also U$1.MECH1, U$1.MECH2, U$2.MECH1, U$2.MECH2, U$3.MECH1, U$3.MECH2, U$4.MECH1, U$4.MECH2
Other:
- board size 25.4 x 13 mm -> 24.3 x 13 mm
- board text added: "BlueRobotics"
Changed lines of the file:
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@@
 <?xml version="1.0" encoding="utf-8"?>
 <!DOCTYPE eagle SYSTEM "eagle.dtd">
-<eagle version="7.6.0">
+<eagle version="7.4.0">
 <drawing>
 <settings>
@@
 <board>
 <plain>
-<wire x1="0" y1="-0.15875" x2="25.38" y2="-0.15875" width="0" layer="20"/>
-<wire x1="25.38" y1="-0.15875" x2="25.38" y2="12.84625" width="0" layer="20"/>
-<wire x1="25.38" y1="12.84625" x2="0" y2="12.84625" width="0" layer="20"/>
-<wire x1="0" y1="12.84625" x2="0" y2="-0.15875" width="0" layer="20"/>
-<text x="4.92125" y="11.1125" size="1.524" layer="25" ratio="12">LEAK</text>
-<text x="14.9225" y="3.81" size="0.635" layer="26" ratio="12" rot="MR0">rev1</text>
-<text x="16.1925" y="0.635" size="0.635" layer="26" ratio="12" rot="MR0">A.S. 8/16</text>
-<text x="24.765" y="8.89" size="1.27" layer="26" ratio="12" rot="MR0">SOS Leak Sensor
+<wire x1="0.635" y1="-0.15875" x2="24.90375" y2="-0.15875" width="0" layer="20"/>
+<wire x1="24.90375" y1="-0.15875" x2="24.90375" y2="12.84625" width="0" layer="20"/>
+<wire x1="24.90375" y1="12.84625" x2="0.635" y2="12.84625" width="0" layer="20"/>
+<wire x1="0.635" y1="12.84625" x2="0.635" y2="-0.15875" width="0" layer="20"/>
+<text x="5.3260625" y="10.9855" size="1.397" layer="25" ratio="12">LEAK</text>
+<text x="24.145875" y="7.699375" size="0.635" layer="26" ratio="12" rot="MR0">rev1</text>
+<text x="5.9769375" y="0.6985" size="0.635" layer="26" ratio="12" rot="MR0">A.S. 8/16</text>
+<text x="24.13" y="8.89" size="1.27" layer="26" ratio="12" rot="MR0">SOS Leak Sensor
 Probe Host Board</text>
 <text x="4.1275" y="10.00125" size="0.8128" layer="25" ratio="12" rot="SR270">GND</text>
 <text x="4.1275" y="7.3025" size="0.8128" layer="25" ratio="12" rot="SR270">+5V</text>
-<text x="0.9525" y="0.9525" size="1.016" layer="21" ratio="12">LEAK</text>
-<wire x1="0.9525" y1="2.2225" x2="4.445" y2="2.2225" width="0.127" layer="21"/>
+<text x="1.3425" y="0.970234375" size="0.8128" layer="21" ratio="12">LEAK</text>
+<wire x1="1.377953125" y1="1.947603125" x2="4.10818125" y2="1.947603125" width="0.127" layer="21"/>
+<text x="6.19125" y="8.5725" size="0.8128" layer="26" ratio="12" rot="SMR0">GND</text>
+<text x="6.19125" y="5.87375" size="0.8128" layer="26" ratio="12" rot="SMR0">+5V</text>
+<text x="6.969125" y="3.33375" size="0.8128" layer="22" ratio="12" rot="MR0">LEAK</text>
+<wire x1="4.1671875" y1="4.3259375" x2="6.9770625" y2="4.3259375" width="0.127" layer="22"/>
+<text x="21.3915625" y="1.6748125" size="1.016" layer="22" ratio="12" rot="MR0">BlueRobotics</text>
 </plain>
 <attributes>
@@
 </autorouter>
 <elements>
-<element name="U$7" library="BR-Eagle-Library" package="BR-LOGO-SMALL" value="LOGOBR-LOGO-S" x="24.4475" y="0.9525" rot="MR0"/>
+<element name="U$7" library="BR-Eagle-Library" package="BR-LOGO-SMALL" value="LOGOBR-LOGO-S" x="24.28875" y="0.9525" rot="MR0"/>
 <element name="R2" library="resistor" package="R0603" value="12K" x="6.35" y="2.2225" rot="R270"/>
 <element name="R1" library="resistor" package="R0603" value="10K" x="9.525" y="7.9375"/>
@@
 <contactref element="U$2" pad="2"/>
 <contactref element="U$3" pad="2"/>
-<contactref element="D1" pad="P$2"/>
 <contactref element="U$4" pad="2"/>
-<polygon width="0.4064" layer="16" isolate="0.3048">
+<polygon width="0.4064" layer="16" isolate="0.3048" thermals="no">
 <vertex x="-1.27" y="13.97"/>
 <vertex x="26.67" y="13.97"/>
@@
 <vertex x="-1.27" y="-1.27"/>
 </polygon>
-<polygon width="0.4064" layer="1" isolate="0.3048">
+<polygon width="0.4064" layer="1" isolate="0.3048" thermals="no">
 <vertex x="-3.81" y="13.97"/>
 <vertex x="-3.81" y="-1.27"/>
@@
 <vertex x="26.67" y="13.97"/>
 </polygon>
-<via x="10.795" y="10.16" extent="1-16" drill="0.6"/>
+<via x="10.4695625" y="10.207625" extent="1-16" drill="0.6"/>
 <via x="12.3825" y="6.35" extent="1-16" drill="0.6"/>
 <via x="18.0975" y="7.9375" extent="1-16" drill="0.6"/>
 <via x="18.0975" y="5.3975" extent="1-16" drill="0.6"/>
-<via x="24.13" y="6.35" extent="1-16" drill="0.6"/>
+<via x="23.495" y="6.35" extent="1-16" drill="0.6"/>
 <contactref element="JP1" pad="1"/>
+<contactref element="U$1" pad="MECH1"/>
+<contactref element="U$1" pad="MECH2"/>
+<contactref element="U$4" pad="MECH1"/>
+<contactref element="U$4" pad="MECH2"/>
+<contactref element="U$3" pad="MECH1"/>
+<contactref element="U$3" pad="MECH2"/>
+<contactref element="U$2" pad="MECH1"/>
+<contactref element="U$2" pad="MECH2"/>
+<contactref element="D1" pad="P$2"/>
 </signal>
 <signal name="SIGNAL">
