File: SOS-Water-Ingress-Sensor.brd (EAGLE design)
At the start: 25.4 x 13 mm, 12 parts

Commit message: Updated pull-down resistor to 2.2k.
Parts:
- R3: value 10K -> 2.2K
Changed lines of the file:
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@@
 <element name="U$1" library="BlueRobotics-JST-GH" package="JST-GH-TOP-2" value="JSH-GH-2VERT" x="14.2875" y="5.23875"/>
 <element name="Q1" library="SparkFun-DiscreteSemi" package="SOT23-3" value="" x="9.525" y="2.2225" rot="R270"/>
-<element name="R3" library="resistor" package="R0603" value="10K" x="9.525" y="5.08" rot="R180"/>
+<element name="R3" library="resistor" package="R0603" value="2.2K" x="9.525" y="5.08" rot="R180"/>
 <element name="U$2" library="BlueRobotics-JST-GH" package="JST-GH-TOP-2" value="JSH-GH-2VERT" x="20.6375" y="5.23875"/>
 <element name="U$3" library="BlueRobotics-JST-GH" package="JST-GH-TOP-2" value="JSH-GH-2VERT" x="15.5575" y="7.46125" rot="R180"/>
